File: Hardware/Modular-Robot-Main/Modular-Robot-Main.kicad_pcb (KiCad board)
At the start: 2 copper layers, 1 part, among them U1 ESP32-S3-WROOM-1

Commit message: Updated pcb and schematic
Parts:
- added J1: USB_C_Receptacle_USB2.0_14P, Connector_USB:USB_C_Receptacle_GCT_USB4110, F.Cu at (38.1, 52.1)
- added J2: Battery, Connector_JST:JST_PH_B2B-PH-K_1x02_P2.00mm_Vertical, F.Cu at (221.0, 35.6)
- added J3: I2c_Front, Connector_PinHeader_2.54mm:PinHeader_1x06_P2.54mm_Horizontal, F.Cu at (222.2, 64.8)
- added J4: I2C_Front_Left, Connector_PinHeader_2.54mm:PinHeader_1x06_P2.54mm_Horizontal, F.Cu at (222.2, 87.6)
- added J5: I2C_Front_Right, Connector_PinHeader_2.54mm:PinHeader_1x06_P2.54mm_Horizontal, F.Cu at (222.2, 113.0)
- added J6: I2C_Back, Connector_PinHeader_2.54mm:PinHeader_1x06_P2.54mm_Horizontal, F.Cu at (252.7, 115.6)
- added J7: I2C_Back_Right, Connector_PinHeader_2.54mm:PinHeader_1x06_P2.54mm_Horizontal, F.Cu at (254.0, 88.9)
- added J8: I2C_Back_Left, Connector_PinHeader_2.54mm:PinHeader_1x06_P2.54mm_Horizontal, F.Cu at (255.3, 67.3)
- added SW1: SW_Push, Button_Switch_SMD:SW_Push_1P1T_NO_CK_KSC6xxJ, F.Cu at (109.2, 59.7)
